File: kicad/voltage_processor.kicad_pcb (KiCad board)
At the start: 2 copper layers, 113 x 110 mm, 222 parts, among them IC1 DG212BDY, IC2 DG212BDY, IC3 DG212BDY, IC4 DG212BDY, J1 ATNVRT_IN_BOTTOM, J10 OUTPUT, J11 CROSSFADE_CV, J12 CROSSFADE_A, J13 CROSSFADE_B, J14 OUTPUT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

Commit message: fixes
Parts:
- moved J11 0.11 mm to (123.1, 128.3)
- moved J12 0.11 mm to (123.1, 106.5)
- moved J13 0.11 mm to (123.1, 117.4)
- moved J7 0.09 mm to (123.1, 69.9)
- moved J8 0.09 mm to (123.1, 48.2)
- moved J9 0.09 mm to (123.1, 59.1)
