File: kicad/voltage_processor_section.kicad_sch (KiCad schematic)
At the start: 105 parts, among them IC1 DG212BDY, IC2 DG212BDY, J10 OUTPUT, J2 ATNVRT_IN_BOTTOM, J7 CROSSFADE_CV, J8 CROSSFADE_A, J9 CROSSFADE_B, Q3 3906, Q4 3904, U1 OPA4134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

Commit message: fixes
Other:
- moved on the sheet: CRSFD1, OFFSET1, R12, R25, R76, R96
